File: eagle/RFID1284/RFID1284.brd (EAGLE design)
At the start: 10 parts

Commit message: Updates to Drawings
Continued Work on Schematic and PCB
Parts:
- added C7: (no value), rcl:C025-040X050
- added C8: (no value), rcl:E2,5-7
- added C9: 100nF, SparkFun:0805
- added IC4: (no value), SparkFun:TO220-IGO
- added J1: POWER_JACKSLT, SparkFun:POWER_JACK_SLOT
- added R1: 10kΩ, SparkFun:0805
- added S1: (no value), SparkFun:TACTILE_SWITCH_SMD
- C1, C2: value (none) -> 20pF; device rcl:C025-040X050 -> SparkFun:0805
- Q2: value (none) -> 16MHz
- moved C6 143.2 mm to (53.3, 24.1)
- moved C4 129.1 mm to (20.3, 34.3)
- moved C5 126.2 mm to (43.2, 17.8)
- moved C1 118.5 mm to (74.9, 11.4)
- moved C2 118.1 mm to (67.3, 11.4)
- moved Q2 114.2 mm to (71.1, 19.1)
- moved C3 104.7 mm to (31.8, 11.4)
- moved IC3 94.6 mm to (22.9, 44.5)
- moved IC1 81.5 mm to (66.0, 41.9)
- moved IC2 68.7 mm to (27.9, 25.4)
Connections:
- removed net N$5: C3.1, IC2.IN
- new net N$4: IC1.9, R1.1, S1.1
- new net N$6: C8.+, IC4.OUT
- new net VIN: C3.1, C4.1, C7.1, IC2.IN, IC3.IN, IC4.IN, J1.PWR
- net 5V: now also R1.2; no longer IC1.32
- net GND: now also C1.1, C2.1, C5.-, C6.-, C7.2, C8.-, C9.1, IC1.11, IC1.31, IC4.GND, J1.GND@1, J1.GND@2, S1.3; no longer C1.2, C2.2
- net N$1: now also C2.2; no longer C2.1
- net N$2: now also C9.2, IC1.32; no longer C4.1, IC3.IN
- net N$3: now also C1.2; no longer C1.1
Other:
- board outline added: 7.1 x 7.3 mm
Changed lines of the file:
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@@
 </autorouter>
 <elements>
-<element name="IC1" library="1284p" package="DIL40" value="" x="16.51" y="-22.86"/>
-<element name="IC2" library="SparkFun" package="TO220-IGO" value="" x="-1.27" y="-36.83"/>
-<element name="IC3" library="SparkFun" package="TO220-IGO" value="" x="-1.27" y="-46.99"/>
-<element name="Q2" library="special" package="QS" value="" x="-5.08" y="-66.04"/>
-<element name="C1" library="rcl" package="C025-040X050" value="" x="-8.89" y="-72.39"/>
-<element name="C2" library="rcl" package="C025-040X050" value="" x="-8.89" y="-78.74"/>
-<element name="C3" library="rcl" package="C025-040X050" value="" x="-8.89" y="-85.09"/>
-<element name="C4" library="rcl" package="C025-040X050" value="" x="-8.89" y="-91.44"/>
-<element name="C5" library="rcl" package="E2,5-7" value="" x="-7.62" y="-97.79"/>
-<element name="C6" library="rcl" package="E2,5-7" value="" x="-7.62" y="-105.41"/>
+<element name="IC1" library="1284p" package="DIL40" value="" x="66.04" y="41.91"/>
+<element name="IC2" library="SparkFun" package="TO220-IGO" value="" x="27.94" y="25.4"/>
+<element name="IC3" library="SparkFun" package="TO220-IGO" value="" x="22.86" y="44.45"/>
+<element name="Q2" library="special" package="QS" value="16MHz" x="71.12" y="19.05"/>
+<element name="C3" library="rcl" package="C025-040X050" value="" x="31.75" y="11.43"/>
+<element name="C4" library="rcl" package="C025-040X050" value="" x="20.32" y="34.29"/>
+<element name="C5" library="rcl" package="E2,5-7" value="" x="43.18" y="17.78"/>
+<element name="C6" library="rcl" package="E2,5-7" value="" x="53.34" y="24.13"/>
+<element name="IC4" library="SparkFun" package="TO220-IGO" value="" x="21.59" y="64.77"/>
+<element name="C7" library="rcl" package="C025-040X050" value="" x="17.78" y="53.34"/>
+<element name="C8" library="rcl" package="E2,5-7" value="" x="52.07" y="59.69"/>
+<element name="R1" library="SparkFun" package="0805" value="10kΩ" x="87.63" y="26.67"/>
+<element name="S1" library="SparkFun" package="TACTILE_SWITCH_SMD" value="" x="87.63" y="19.05"/>
+<element name="C1" library="SparkFun" package="0805" value="20pF" x="74.93" y="11.43"/>
+<element name="C2" library="SparkFun" package="0805" value="20pF" x="67.31" y="11.43"/>
+<element name="J1" library="SparkFun" package="POWER_JACK_SLOT" value="POWER_JACKSLT" x="66.04" y="58.42"/>
+<element name="C9" library="SparkFun" package="0805" value="100nF" x="71.12" y="54.61"/>
 </elements>
 <signals>
@@
 <contactref element="IC2" pad="GND"/>
 <contactref element="IC3" pad="GND"/>
-<contactref element="C1" pad="2"/>
-<contactref element="C2" pad="2"/>
 <contactref element="C4" pad="2"/>
 <contactref element="C3" pad="2"/>
-<wire x1="-7.62" y1="-85.09" x2="-7.62" y2="-91.44" width="0" layer="19" extent="1-1"/>
-<wire x1="-7.62" y1="-78.74" x2="-7.62" y2="-85.09" width="0" layer="19" extent="1-1"/>
-<wire x1="-7.62" y1="-72.39" x2="-7.62" y2="-78.74" width="0" layer="19" extent="1-1"/>
-<wire x1="-1.27" y1="-46.99" x2="-7.62" y2="-72.39" width="0" layer="19" extent="1-1"/>
-<wire x1="-1.27" y1="-36.83" x2="-1.27" y2="-46.99" width="0" layer="19" extent="1-1"/>
+<contactref element="C5" pad="-"/>
+<contactref element="C6" pad="-"/>
+<contactref element="C8" pad="-"/>
+<contactref element="IC4" pad="GND"/>
+<contactref element="C7" pad="2"/>
+<contactref element="IC1" pad="31"/>
+<contactref element="IC1" pad="11"/>
+<contactref element="S1" pad="3"/>
+<contactref element="C1" pad="1"/>
+<contactref element="C2" pad="1"/>
+<contactref element="J1" pad="GND@1"/>
+<contactref element="J1" pad="GND@2"/>
+<contactref element="C9" pad="1"/>
+<wire x1="68.62" y1="65.92" x2="73.62" y2="69.22" width="0" layer="19" extent="1-1"/>
+<wire x1="70.22" y1="54.61" x2="68.62" y2="65.92" width="0" layer="19" extent="1-1"/>
+<wire x1="64.77" y1="49.53" x2="70.22" y2="54.61" width="0" layer="19" extent="1-1"/>
+<wire x1="53.34" y1="59.69" x2="64.77" y2="49.53" width="0" layer="19" extent="1-1"/>
+<wire x1="67.31" y1="34.29" x2="64.77" y2="49.53" width="0" layer="19" extent="1-1"/>
+<wire x1="54.61" y1="24.13" x2="67.31" y2="34.29" width="0" layer="19" extent="1-1"/>
+<wire x1="44.45" y1="17.78" x2="54.61" y2="24.13" width="0" layer="19" extent="1-1"/>
+<wire x1="33.02" y1="11.43" x2="44.45" y2="17.78" width="0" layer="19" extent="1-1"/>
+<wire x1="27.94" y1="25.4" x2="33.02" y2="11.43" width="0" layer="19" extent="1-1"/>
+<wire x1="21.59" y1="34.29" x2="27.94" y2="25.4" width="0" layer="19" extent="1-1"/>
+<wire x1="22.86" y1="44.45" x2="21.59" y2="34.29" width="0" layer="19" extent="1-1"/>
+<wire x1="19.05" y1="53.34" x2="22.86" y2="44.45" width="0" layer="19" extent="1-1"/>
+<wire x1="21.59" y1="64.77" x2="19.05" y2="53.34" width="0" layer="19" extent="1-1"/>
+<wire x1="66.41" y1="11.43" x2="54.61" y2="24.13" width="0" layer="19" extent="1-1"/>
+<wire x1="74.03" y1="11.43" x2="66.41" y2="11.43" width="0" layer="19" extent="1-1"/>
+<wire x1="85.09" y1="17.145" x2="74.03" y2="11.43" width="0" layer="19" extent="1-1"/>
 </signal>
 <signal name="5V">
-<contactref element="IC1" pad="32"/>
 <contactref element="IC1" pad="30"/>
 <contactref element="IC1" pad="10"/>
 <contactref element="IC2" pad="OUT"/>
 <contactref element="C5" pad="+"/>
-<wire x1="1.27" y1="-36.83" x2="-8.89" y2="-97.79" width="0" layer="19" extent="1-1"/>
-<wire x1="15.24" y1="-30.48" x2="1.27" y2="-36.83" width="0" layer="19" extent="1-1"/>
-<wire x1="12.7" y1="-15.24" x2="15.24" y2="-30.48" width="0" layer="19" extent="1-1"/>
-<wire x1="17.78" y1="-15.24" x2="12.7" y2="-15.24" width="0" layer="19" extent="1-1"/>
+<contactref element="R1" pad="2"/>
+<wire x1="64.77" y1="34.29" x2="67.31" y2="49.53" width="0" layer="19" extent="1-1"/>
+<wire x1="88.53" y1="26.67" x2="64.77" y2="34.29" width="0" layer="19" extent="1-1"/>
+<wire x1="41.91" y1="17.78" x2="64.77" y2="34.29" width="0" layer="19" extent="1-1"/>
+<wire x1="30.48" y1="25.4" x2="41.91" y2="17.78" width="0" layer="19" extent="1-1"/>
 </signal>
 <signal name="N$3">
 <contactref element="IC1" pad="13"/>
 <contactref element="Q2" pad="2"/>
-<contactref element="C1" pad="1"/>
-<wire x1="-2.54" y1="-66.04" x2="-10.16" y2="-72.39" width="0" layer="19" extent="1-1"/>
-<wire x1="22.86" y1="-30.48" x2="-2.54" y2="-66.04" width="0" layer="19" extent="1-1"/>
+<contactref element="C1" pad="2"/>
+<wire x1="73.66" y1="19.05" x2="72.39" y2="34.29" width="0" layer="19" extent="1-1"/>
+<wire x1="75.83" y1="11.43" x2="73.66" y2="19.05" width="0" layer="19" extent="1-1"/>
 </signal>
 <signal name="N$1">
 <contactref element="IC1" pad="12"/>
 <contactref element="Q2" pad="1"/>
-<contactref element="C2" pad="1"/>
-<wire x1="-7.62" y1="-66.04" x2="-10.16" y2="-78.74" width="0" layer="19" extent="1-1"/>
-<wire x1="20.32" y1="-30.48" x2="-7.62" y2="-66.04" width="0" layer="19" extent="1-1"/>
+<contactref element="C2" pad="2"/>
+<wire x1="68.58" y1="19.05" x2="69.85" y2="34.29" width="0" layer="19" extent="1-1"/>
+<wire x1="68.21" y1="11.43" x2="68.58" y2="19.05" width="0" layer="19" extent="1-1"/>
 </signal>
-<signal name="N$2">
+<signal name="VIN">
+<contactref element="C3" pad="1"/>
+<contactref element="IC2" pad="IN"/>
 <contactref element="C4" pad="1"/>
 <contactref element="IC3" pad="IN"/>
-<wire x1="-3.81" y1="-46.99" x2="-10.16" y2="-91.44" width="0" layer="19" extent="1-1"/>
-</signal>
-<signal name="N$5">
-<contactref element="C3" pad="1"/>
-<contactref element="IC2" pad="IN"/>
-<wire x1="-3.81" y1="-36.83" x2="-10.16" y2="-85.09" width="0" layer="19" extent="1-1"/>
+<contactref element="C7" pad="1"/>
+<contactref element="IC4" pad="IN"/>
+<contactref element="J1" pad="PWR"/>
+<wire x1="19.05" y1="64.77" x2="68.62" y2="72.22" width="0" layer="19" extent="1-1"/>
+<wire x1="16.51" y1="53.34" x2="19.05" y2="64.77" width="0" layer="19" extent="1-1"/>
+<wire x1="20.32" y1="44.45" x2="16.51" y2="53.34" width="0" layer="19" extent="1-1"/>
+<wire x1="19.05" y1="34.29" x2="20.32" y2="44.45" width="0" layer="19" extent="1-1"/>
+<wire x1="25.4" y1="25.4" x2="19.05" y2="34.29" width="0" layer="19" extent="1-1"/>
+<wire x1="30.48" y1="11.43" x2="25.4" y2="25.4" width="0" layer="19" extent="1-1"/>
 </signal>
 <signal name="VCC">
 <contactref element="IC3" pad="OUT"/>
 <contactref element="C6" pad="+"/>
-<wire x1="1.27" y1="-46.99" x2="-8.89" y2="-105.41" width="0" layer="19" extent="1-1"/>
+<wire x1="25.4" y1="44.45" x2="52.07" y2="24.13" width="0" layer="19" extent="1-1"/>
+</signal>
+<signal name="N$6">
+<contactref element="IC4" pad="OUT"/>
+<contactref element="C8" pad="+"/>
+<wire x1="24.13" y1="64.77" x2="50.8" y2="59.69" width="0" layer="19" extent="1-1"/>
+</signal>
+<signal name="N$4">
+<contactref element="R1" pad="1"/>
+<contactref element="IC1" pad="9"/>
+<contactref element="S1" pad="1"/>
+<wire x1="85.09" y1="20.955" x2="86.73" y2="26.67" width="0" layer="19" extent="1-1"/>
+<wire x1="62.23" y1="34.29" x2="86.73" y2="26.67" width="0" layer="19" extent="1-1"/>
+</signal>
+<signal name="N$2">
+<contactref element="IC1" pad="32"/>
+<contactref element="C9" pad="2"/>
+<wire x1="62.23" y1="49.53" x2="72.02" y2="54.61" width="0" layer="19" extent="1-1"/>
 </signal>
 </signals>
