File: eagle/RFID1284/RFID1284.sch (EAGLE design)
At the start: 10 parts

Commit message: Updates to Drawings
Continued Work on Schematic and PCB
Parts:
- added C7: (no value), rcl:C-US025-040X050
- added C8: (no value), rcl:CPOL-USE2.5-7
- added C9: 100nF, SparkFun:CAP0805
- added IC4: (no value), SparkFun:V_REG_78XXSINK
- added J1: POWER_JACKSLT, SparkFun:POWER_JACKSLT
- added R1: 10kΩ, SparkFun:RESISTOR0805-RES
- added S1: (no value), SparkFun:TAC_SWITCHSMD
- C1, C2: value (none) -> 20pF; device rcl:C-US025-040X050 -> SparkFun:CAP0805
- Q2: value (none) -> 16MHz
Connections:
- removed net N$5: C3.1, IC2.IN
- new net N$4: IC1.RESET, R1.1, S1.1
- new net N$6: C8.+, IC4.OUT
- new net VIN: C3.1, C4.1, C7.1, IC2.IN, IC3.IN, IC4.IN, J1.PWR
- net 5V: now also R1.2; no longer IC1.AREF
- net GND: now also C1.1, C2.1, C5.-, C6.-, C7.2, C8.-, C9.1, IC1.GND@0, IC1.GND@1, IC4.GND, J1.GND, J1.GNDBREAK, S1.3; no longer C1.2, C2.2
- net N$1: now also C2.2; no longer C2.1
- net N$2: now also C9.2, IC1.AREF; no longer C4.1, IC3.IN
- net N$3: now also C1.2; no longer C1.1
Other:
- moved on the sheet: C1, C2

Commit message: Kind of Done
Parts:
- removed C2: 20pF, SparkFun:CAP0805
- removed C9: 100nF, SparkFun:CAP0805
- added J2: AVR_SPI_PRG_6NS, SparkFun:AVR_SPI_PRG_6NS
- added JP1, JP2, JP3, JP6: (no value), SparkFun:M04LOCK_LONGPADS
- added JP4: (no value), SparkFun:M02LOCK_LONGPADS
- added JP5: (no value), SparkFun:M06LOCK_LONGPADS
- added JP7: (no value), SparkFun:M08LOCK_LONGPADS
- added JP8: (no value), SparkFun:M04LONGPADS
- added Q1: (no value), SparkFun:TRANSISTOR_NPNTO-92-AMMO
- added R4: 10kΩ, SparkFun:RESISTORPTH-1/4W
- added R5: 8.2kΩ, SparkFun:RESISTORPTH-1/4W
- added R6: 12kΩ, SparkFun:RESISTORPTH-1/4W
- added SERVO: (no value), SparkFun:M03LONGPADS
- added U$4: XBEE-1B1, SparkFun:XBEE-1B1
- C1: value 20pF -> 100nF; device SparkFun:CAP0805 -> SparkFun:CAPPTH1
- C7: value (none) -> 20pF; device rcl:C-US025-040X050 -> SparkFun:CAPPTH1
- C8: value (none) -> 20pF; device rcl:CPOL-USE2.5-7 -> SparkFun:CAPPTH1
- R1: value 10kΩ -> (none); device SparkFun:RESISTOR0805-RES -> SparkFun:RESISTORPTH-1/4W
- S1: device SparkFun:TAC_SWITCHSMD -> SparkFun:TAC_SWITCHPTH
Connections:
- removed net N$4: IC1.RESET, R1.1, S1.1
- new net DOOR_SWITCH: IC1.T1/CLK0/PCINT9, JP4.1
- new net LOCK: IC1.AIN0/INT2/PCINT10, JP2.1
- new net LOCK_DELAY: IC1.AIN1/OC0A/PCINT11, JP3.1
- new net MISO: IC1.MISO/OC3A/PCINT14, J2.1, JP6.3
- new net MOSI: IC1.MOSI/ICP3/PCINT13, J2.4, JP6.2
- new net N$10: IC1.ADC3/PCINT3, JP5.2
- new net N$11: IC1.ADC4/PCINT4, JP5.3
- new net N$12: IC1.ADC5/PCINT5, JP5.4
- new net N$13: IC1.ADC6/PCINT6, JP5.5
- new net N$14: IC1.ADC7/PCINT7, JP5.6
- new net N$19: IC1.SCL/PCINT16, JP7.1
- new net N$20: IC1.SDA/PCINT17, JP7.2
- new net N$21: IC1.TCK/PCINT18, JP7.3
- new net N$22: IC1.TMS/PCINT19, JP7.4
- new net N$23: IC1.TDO/PCINT20, JP7.5
- new net N$24: IC1.TDI/PCINT21, JP7.6
- new net N$25: IC1.TOSC1/PCINT22, JP7.7
- new net N$26: IC1.TOSC2/PCINT23, JP7.8
- new net RELAY_RESET: IC1.ADC1/PCINT1
- new net RELAY_SET: IC1.ADC0/PCINT0
- new net RESET: IC1.RESET, J2.5, R4.1, S1.1
- new net RFID_ENABLE: IC1.OC2A/PCINT31, JP8.3
- new net RFID_SERIAL: IC1.RXD1/INT0/PCINT26, JP8.2
- new net SCK: IC1.SCK/OC3B/PCINT15, J2.3, JP6.4
- new net SERVO: IC1.OC1A/PCINT29, Q1.B
- new net SERVO_OUT: Q1.E, R1.2, SERVO.1
- new net SERVO_VCC: C6.+, IC3.OUT, SERVO.2
- new net SS: IC1.SS/OC0B/PCINT12, JP6.1
- new net TX0: IC1.TXD0/PCINT25, R5.1
- new net TX0_LOW: R5.2, R6.1, U$4.DIN
- new net UNLOCK: IC1.T0/XCK0/PCINT8, JP1.1
- new net XBEE_OUT: IC1.T3/RXD0/PCINT24, U$4.DOUT
- net 5V: now also IC4.OUT, J2.2, JP1.3, JP2.3, JP3.3, JP8.4, Q1.C, R4.2; no longer R1.2
- net GND: now also C7.1, C8.1, IC4.IN, J2.6, JP1.2, JP1.4, JP2.2, JP2.4, JP3.2, JP3.4, JP4.2, JP8.1, R1.1, R6.2, SERVO.3, U$4.GND; no longer C2.1, C7.2, C8.-, C9.1, IC4.GND
- net N$1: now also C7.2; no longer C2.2
- net N$2: now also C1.2; no longer C9.2
- net N$3: now also C8.2; no longer C1.2
- net N$6: now also IC1.ADC2/PCINT2, JP5.1; no longer C8.+, IC4.OUT
- net VCC: now also IC4.GND, U$4.VDD; no longer C6.+, IC3.OUT
- net VIN: no longer C7.1, IC4.IN
Other:
- moved on the sheet: C1, C7, R1
